File: active.sch (KiCad schematic (older format))
At the start: 32 parts, among them P1 CONN_1, P10 CONN_1, P11 CONN_1, P2 CONN_1, P3 CONN_1, P4 CONN_1, P5 CONN_1, P6 CONN_1, P7 CONN_1, P8 SPI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

Commit message: fixed LED positions, added svg export, added copyright info and oshw logo to the pcb
Changed lines of the file:
@@
-EESchema Schematic File Version 2  date Thu 09 Feb 2012 10:18:34 AM CET
+EESchema Schematic File Version 2  date Fri 10 Feb 2012 10:08:11 AM CET
 LIBS:power
 LIBS:device
@@
 Sheet 1 1
 Title ""
-Date "30 dec 2011"
+Date "10 feb 2012"
 Rev ""
 Comp ""
@@
 Comment4 ""
 $EndDescr
+Text Label 6700 2100 0    60   ~ 0
+vaa
+Text Label 6700 2000 0    60   ~ 0
+agnd
+Text Label 6700 1900 0    60   ~ 0
+vdd
+Text Label 6700 1800 0    60   ~ 0
+gnd
+Wire Wire Line
+	6650 2000 6750 2000
 Wire Wire Line
 	6650 1800 6750 1800
@@
 Wire Wire Line
 	4100 2400 4100 2550
+Wire Wire Line
+	6650 1900 6750 1900
 Text Label 4100 2550 0    60   ~ 0
 ref
@@
 L AGND #PWR18
 U 1 1 4EFCC87D
-P 6750 2000
-F 0 "#PWR18" H 6750 2000 40  0001 C CNN
-F 1 "AGND" H 6750 1930 50  0000 C CNN
-	1    6750 2000
+P 6650 2000
+F 0 "#PWR18" H 6650 2000 40  0001 C CNN
+F 1 "AGND" H 6650 1930 50  0000 C CNN
+	1    6650 2000
 	0    1    1    0
 $EndComp
@@
 L VDD #PWR17
 U 1 1 4EFCC86C
-P 6750 1900
-F 0 "#PWR17" H 6750 2000 30  0001 C CNN
-F 1 "VDD" H 6750 2010 30  0000 C CNN
-	1    6750 1900
-	0    -1   -1   0
-$EndComp
+P 6650 1900
+F 0 "#PWR17" H 6650 2000 30  0001 C CNN
+F 1 "VDD" H 6650 2010 30  0000 C CNN
+	1    6650 1900
+	0    -1   -1   0
+$EndComp
