File: active.sch (KiCad schematic (older format))
At the start: 32 parts, among them P1 CONN_1, P10 CONN_1, P11 CONN_1, P2 CONN_1, P3 CONN_1, P4 CONN_1, P5 CONN_1, P6 CONN_1, P7 CONN_1, P8 SPI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

Commit message: Added some doc
Parts:
- added P12: CONN_1, symbol CONN_1
Connections:
- net at C8.2, R10.1, U1.28 (RLDINV): now also P12.1
Changed lines of the file:
@@
-EESchema Schematic File Version 2  date Thu 16 Feb 2012 11:20:04 AM CET
+EESchema Schematic File Version 2  date Thu 16 Feb 2012 12:05:28 PM CET
 LIBS:power
 LIBS:device
@@
 Sheet 1 1
 Title ""
-Date "10 feb 2012"
+Date "16 feb 2012"
 Rev ""
 Comp ""
@@
 Comment4 ""
 $EndDescr
+$Comp
+L CONN_1 P12
+U 1 1 4F3CE2EB
+P 4800 1750
+F 0 "P12" H 4880 1750 40  0000 L CNN
+F 1 "CONN_1" H 4800 1805 30  0001 C CNN
+	1    4800 1750
+	0    -1   -1   0
+$EndComp
 Text Label 6700 2100 0    60   ~ 0
 vaa
@@
 $EndComp
 $Comp
-L VAA #PWR16
+L VAA #PWR18
 U 1 1 4EFCC8CB
 P 6700 2100
-F 0 "#PWR16" H 6700 2160 30  0001 C CNN
+F 0 "#PWR18" H 6700 2160 30  0001 C CNN
 F 1 "VAA" H 6700 2210 30  0000 C CNN
 	1    6700 2100
@@
 $EndComp
 $Comp
-L AGND #PWR18
+L AGND #PWR17
 U 1 1 4EFCC87D
 P 6650 2000
-F 0 "#PWR18" H 6650 2000 40  0001 C CNN
+F 0 "#PWR17" H 6650 2000 40  0001 C CNN
 F 1 "AGND" H 6650 1930 50  0000 C CNN
 	1    6650 2000
@@
 $EndComp
 $Comp
-L VDD #PWR17
+L VDD #PWR16
 U 1 1 4EFCC86C
 P 6650 1900
-F 0 "#PWR17" H 6650 2000 30  0001 C CNN
+F 0 "#PWR16" H 6650 2000 30  0001 C CNN
 F 1 "VDD" H 6650 2010 30  0000 C CNN
 	1    6650 1900

Commit message: small clarification in the schmematic
Other:
- moved on the sheet: P10, R10, R9
Changed lines of the file:
@@
-EESchema Schematic File Version 2  date Thu 16 Feb 2012 12:05:28 PM CET
+EESchema Schematic File Version 2  date Thu 16 Feb 2012 12:25:49 PM CET
 LIBS:power
 LIBS:device
@@
 	5000 2600 5000 1900
 Wire Wire Line
-	5000 1900 4600 1900
+	5000 1900 4800 1900
 Wire Wire Line
-	4600 2400 4800 2400
+	4800 1900 4450 1900
+Wire Wire Line
+	4450 2400 4800 2400
 Wire Wire Line
 	6750 2100 6700 2100
@@
 Connection ~ 7100 3000
 Wire Wire Line
-	7100 2750 7100 3100
+	7100 2750 7100 3000
+Wire Wire Line
+	7100 3000 7100 3100
 Connection ~ 3700 4000
 Wire Wire Line
-	3700 3900 3700 4100
+	3700 3900 3700 4000
+Wire Wire Line
+	3700 4000 3700 4100
 Wire Wire Line
 	5400 5100 5400 4850
@@
 	4800 1900 4800 2000
 Wire Wire Line
-	4100 2400 4100 2550
+	3950 2400 3800 2400
 Wire Wire Line
 	6650 1900 6750 1900
-Text Label 4100 2550 0    60   ~ 0
+Text Label 3800 2400 0    60   ~ 0
 ref
 $Comp
@@
 L CONN_1 P10
 U 1 1 4EFD05E7
-P 3950 2400
-F 0 "P10" H 4030 2400 40  0000 L CNN
-F 1 "CONN_1" H 3950 2455 30  0001 C CNN
-	1    3950 2400
+P 3650 2400
+F 0 "P10" H 3730 2400 40  0000 L CNN
+F 1 "CONN_1" H 3650 2455 30  0001 C CNN
+	1    3650 2400
 	-1   0    0    1
 $EndComp
@@
 L R R9
 U 1 1 4EFD05B9
-P 4350 2400
-F 0 "R9" V 4430 2400 50  0000 C CNN
-F 1 "20k" V 4350 2400 50  0000 C CNN
-	1    4350 2400
+P 4200 2400
+F 0 "R9" V 4280 2400 50  0000 C CNN
+F 1 "20k" V 4200 2400 50  0000 C CNN
+	1    4200 2400
 	0    1    1    0
 $EndComp
@@
 L R R10
 U 1 1 4EFD043C
-P 4600 2150
-F 0 "R10" V 4680 2150 50  0000 C CNN
-F 1 "1M" V 4600 2150 50  0000 C CNN
-	1    4600 2150
+P 4450 2150
+F 0 "R10" V 4530 2150 50  0000 C CNN
+F 1 "1M" V 4450 2150 50  0000 C CNN
+	1    4450 2150
 	1    0    0    -1
 $EndComp
