File: channel.sch (KiCad schematic (older format))
At the start: 11 parts, among them U2 CA3140, U3 INA155

Commit message: Finished the two-channel dual ti afe/pure analog-arduino adc version.
Changed lines of the file:
@@
-EESchema Schematic File Version 2  date Fri 25 May 2012 04:08:34 PM CEST
+EESchema Schematic File Version 2  date Fri 25 May 2012 10:34:43 PM CEST
 LIBS:power
 LIBS:device
@@
 LIBS:openmind-custom
 LIBS:ti-afe
-LIBS:modular-dual-cache
+LIBS:modular-half-dual-cache
 EELAYER 25  0
 EELAYER END
 $Descr A4 11700 8267
 encoding utf-8
-Sheet 9 11
+Sheet 9 6
 Title ""
 Date "25 may 2012"
@@
 AR Path="/4FB7BCB8/4FBE8C14" Ref="U4"  Part="1"
 AR Path="/4FB7B986/4FBE8C14" Ref="U5"  Part="1"
-F 0 "U2" H 4750 4350 70  0000 C CNN
+F 0 "U5" H 4750 4350 70  0000 C CNN
 F 1 "INA155" H 4850 3850 70  0000 C CNN
 	1    4450 4100
@@
 AR Path="/4FB7BCB8/4FB7BB90" Ref="C14"  Part="1"
 AR Path="/4FB7B986/4FB7BB90" Ref="C17"  Part="1"
-F 0 "C8" H 5200 4200 50  0000 L CNN
+F 0 "C17" H 5200 4200 50  0000 L CNN
 F 1 "1µ" H 5200 4000 50  0000 L CNN
 	1    5150 4100
@@
 AR Path="/4FB7BCB8/4FB7BB8F" Ref="R37"  Part="1"
 AR Path="/4FB7B986/4FB7BB8F" Ref="R45"  Part="1"
-F 0 "R21" V 5880 4100 50  0000 C CNN
+F 0 "R45" V 5880 4100 50  0000 C CNN
 F 1 "2k2" V 5800 4100 50  0000 C CNN
 	1    5800 4100
@@
 AR Path="/4FB7BCB8/4FB7BB8E" Ref="R36"  Part="1"
 AR Path="/4FB7B986/4FB7BB8E" Ref="R44"  Part="1"
-F 0 "R20" V 5530 4450 50  0000 C CNN
+F 0 "R44" V 5530 4450 50  0000 C CNN
 F 1 "1M" V 5450 4450 50  0000 C CNN
 	1    5450 4450
@@
 AR Path="/4FB7BD19/4FB7BB8D" Ref="#PWR031"  Part="1"
 AR Path="/4FB7BCFA/4FB7BB8D" Ref="#PWR035"  Part="1"
-AR Path="/4FB7BCB8/4FB7BB8D" Ref="#PWR039"  Part="1"
-AR Path="/4FB7B986/4FB7BB8D" Ref="#PWR043"  Part="1"
-F 0 "#PWR043" H 5450 4800 40  0001 C CNN
+AR Path="/4FB7BCB8/4FB7BB8D" Ref="#PWR027"  Part="1"
+AR Path="/4FB7B986/4FB7BB8D" Ref="#PWR031"  Part="1"
+F 0 "#PWR031" H 5450 4800 40  0001 C CNN
 F 1 "AGND" H 5450 4730 50  0000 C CNN
 	1    5450 4800
@@
 AR Path="/4FB7BCB8/4FB7BB8C" Ref="R40"  Part="1"
 AR Path="/4FB7B986/4FB7BB8C" Ref="R48"  Part="1"
-F 0 "R24" V 7830 4000 50  0000 C CNN
+F 0 "R48" V 7830 4000 50  0000 C CNN
 F 1 "10k" V 7750 4000 50  0000 C CNN
 	1    7750 4000
@@
 AR Path="/4FB7BCB8/4FB7BB8B" Ref="C16"  Part="1"
 AR Path="/4FB7B986/4FB7BB8B" Ref="C19"  Part="1"
-F 0 "C10" H 8150 4400 50  0000 L CNN
+F 0 "C19" H 8150 4400 50  0000 L CNN
 F 1 "440n" H 8150 4200 50  0000 L CNN
 	1    8100 4300
@@
 AR Path="/4FB7BD19/4FB7BB8A" Ref="#PWR032"  Part="1"
 AR Path="/4FB7BCFA/4FB7BB8A" Ref="#PWR036"  Part="1"
-AR Path="/4FB7BCB8/4FB7BB8A" Ref="#PWR040"  Part="1"
-AR Path="/4FB7B986/4FB7BB8A" Ref="#PWR044"  Part="1"
-F 0 "#PWR044" H 8100 4600 40  0001 C CNN
+AR Path="/4FB7BCB8/4FB7BB8A" Ref="#PWR028"  Part="1"
+AR Path="/4FB7B986/4FB7BB8A" Ref="#PWR032"  Part="1"
+F 0 "#PWR032" H 8100 4600 40  0001 C CNN
 F 1 "AGND" H 8100 4530 50  0000 C CNN
 	1    8100 4600
@@
 AR Path="/4FB7BCB8/4FB7BB89" Ref="C15"  Part="1"
 AR Path="/4FB7B986/4FB7BB89" Ref="C18"  Part="1"
-F 0 "C9" H 6600 3300 50  0000 L CNN
+F 0 "C18" H 6600 3300 50  0000 L CNN
 F 1 "6n8" H 6600 3100 50  0000 L CNN
 	1    6550 3200
@@
 AR Path="/4FB7BCB8/4FB7BB88" Ref="R39"  Part="1"
 AR Path="/4FB7B986/4FB7BB88" Ref="R47"  Part="1"
-F 0 "R23" V 6630 2950 50  0000 C CNN
+F 0 "R47" V 6630 2950 50  0000 C CNN
 F 1 "1M" V 6550 2950 50  0000 C CNN
 	1    6550 2950
@@
 AR Path="/4FB7BD19/4FB7BB86" Ref="#PWR033"  Part="1"
 AR Path="/4FB7BCFA/4FB7BB86" Ref="#PWR037"  Part="1"
-AR Path="/4FB7BCB8/4FB7BB86" Ref="#PWR041"  Part="1"
-AR Path="/4FB7B986/4FB7BB86" Ref="#PWR045"  Part="1"
-F 0 "#PWR045" H 6550 4500 40  0001 C CNN
+AR Path="/4FB7BCB8/4FB7BB86" Ref="#PWR029"  Part="1"
+AR Path="/4FB7B986/4FB7BB86" Ref="#PWR033"  Part="1"
+F 0 "#PWR033" H 6550 4500 40  0001 C CNN
 F 1 "AGND" H 6550 4400 50  0000 C CNN
 	1    6550 4500
@@
 AR Path="/4FB7BD19/4FB7BB85" Ref="#PWR034"  Part="1"
 AR Path="/4FB7BCFA/4FB7BB85" Ref="#PWR038"  Part="1"
-AR Path="/4FB7BCB8/4FB7BB85" Ref="#PWR042"  Part="1"
-AR Path="/4FB7B986/4FB7BB85" Ref="#PWR046"  Part="1"
-F 0 "#PWR046" H 4350 4500 40  0001 C CNN
+AR Path="/4FB7BCB8/4FB7BB85" Ref="#PWR030"  Part="1"
+AR Path="/4FB7B986/4FB7BB85" Ref="#PWR034"  Part="1"
+F 0 "#PWR034" H 4350 4500 40  0001 C CNN
 F 1 "AGND" H 4350 4430 50  0000 C CNN
 	1    4350 4500
@@
 AR Path="/4FB7BCB8/4FB7BB7E" Ref="R35"  Part="1"
 AR Path="/4FB7B986/4FB7BB7E" Ref="R43"  Part="1"
-F 0 "R19" V 4630 4750 50  0000 C CNN
+F 0 "R43" V 4630 4750 50  0000 C CNN
 F 1 "20k" V 4550 4750 50  0000 C CNN
 	1    4550 4750
@@
 AR Path="/4FB7BCB8/4FB7BB7D" Ref="RV5"  Part="1"
 AR Path="/4FB7B986/4FB7BB7D" Ref="RV6"  Part="1"
-F 0 "RV3" H 7200 4300 50  0000 C CNN
+F 0 "RV6" H 7200 4300 50  0000 C CNN
 F 1 "10k" H 7200 4400 50  0000 C CNN
 	1    7200 4400
-	0    -1   -1   0
+	0    -1   1    0
 $EndComp
 $Comp
@@
 AR Path="/4FB7BCB8/4FB7BB7C" Ref="U10"  Part="1"
 AR Path="/4FB7B986/4FB7BB7C" Ref="U12"  Part="1"
-F 0 "U6" H 6650 4000 60  0000 C CNN
+F 0 "U12" H 6650 4000 60  0000 C CNN
 F 1 "CA3140" H 6800 3800 50  0000 C CNN
 	1    6650 4000
