File: input.sch (KiCad schematic (older format))
At the start: 4 parts, among them J3 SMA, J4 SMA

Commit message: Finished the two-channel dual ti afe/pure analog-arduino adc version.
Changed lines of the file:
@@
-EESchema Schematic File Version 2  date Fri 25 May 2012 04:08:34 PM CEST
+EESchema Schematic File Version 2  date Fri 25 May 2012 10:34:43 PM CEST
 LIBS:power
 LIBS:device
@@
 LIBS:openmind-custom
 LIBS:ti-afe
-LIBS:modular-dual-cache
+LIBS:modular-half-dual-cache
 EELAYER 25  0
 EELAYER END
 $Descr A4 11700 8267
 encoding utf-8
-Sheet 2 11
+Sheet 2 6
 Title ""
 Date "25 may 2012"
@@
 AR Path="/4FBE6CF5/4FBE6C5A" Ref="J7"  Part="1"
 AR Path="/4FBE6CE5/4FBE6C5A" Ref="J5"  Part="1"
-F 0 "J3" H 1775 1715 60  0000 C CNN
+F 0 "J5" H 1775 1715 60  0000 C CNN
 F 1 "SMA" H 1840 1640 60  0000 C CNN
 F 2 "SMA" H 1825 1570 50  0000 C CNN
@@
 AR Path="/4FBE6CF5/4FBE6C59" Ref="J8"  Part="1"
 AR Path="/4FBE6CE5/4FBE6C59" Ref="J6"  Part="1"
-F 0 "J4" H 1775 2515 60  0000 C CNN
+F 0 "J6" H 1775 2515 60  0000 C CNN
 F 1 "SMA" H 1840 2440 60  0000 C CNN
 F 2 "SMA" H 1825 2370 50  0000 C CNN
@@
 AR Path="/4FBE6CF5/4FBE6C58" Ref="R60"  Part="1"
 AR Path="/4FBE6CE5/4FBE6C58" Ref="R58"  Part="1"
-F 0 "R56" V 2230 1700 50  0000 C CNN
+F 0 "R58" V 2230 1700 50  0000 C CNN
 F 1 "20k" V 2150 1700 50  0000 C CNN
 	1    2150 1700
@@
 AR Path="/4FBE6CF5/4FBE6C57" Ref="R61"  Part="1"
 AR Path="/4FBE6CE5/4FBE6C57" Ref="R59"  Part="1"
-F 0 "R57" V 2230 1900 50  0000 C CNN
+F 0 "R59" V 2230 1900 50  0000 C CNN
 F 1 "20k" V 2150 1900 50  0000 C CNN
 	1    2150 1900
@@
 $EndComp
 $Comp
-L AGND #PWR019
+L AGND #PWR020
 U 1 1 4FBE6C56
 P 1850 1550
-AR Path="/4FBE6C46/4FBE6C56" Ref="#PWR019"  Part="1"
+AR Path="/4FBE6C46/4FBE6C56" Ref="#PWR020"  Part="1"
 AR Path="/4FBE6CFE/4FBE6C56" Ref="#PWR013"  Part="1"
 AR Path="/4FBE6CF5/4FBE6C56" Ref="#PWR015"  Part="1"
-AR Path="/4FBE6CE5/4FBE6C56" Ref="#PWR017"  Part="1"
-F 0 "#PWR019" H 1850 1550 40  0001 C CNN
+AR Path="/4FBE6CE5/4FBE6C56" Ref="#PWR018"  Part="1"
+F 0 "#PWR020" H 1850 1550 40  0001 C CNN
 F 1 "AGND" H 1850 1480 50  0000 C CNN
 	1    1850 1550
@@
 $EndComp
 $Comp
-L AGND #PWR020
+L AGND #PWR021
 U 1 1 4FBE6C55
 P 1750 2250
-AR Path="/4FBE6C46/4FBE6C55" Ref="#PWR020"  Part="1"
+AR Path="/4FBE6C46/4FBE6C55" Ref="#PWR021"  Part="1"
 AR Path="/4FBE6CFE/4FBE6C55" Ref="#PWR014"  Part="1"
 AR Path="/4FBE6CF5/4FBE6C55" Ref="#PWR016"  Part="1"
-AR Path="/4FBE6CE5/4FBE6C55" Ref="#PWR018"  Part="1"
-F 0 "#PWR020" H 1750 2250 40  0001 C CNN
+AR Path="/4FBE6CE5/4FBE6C55" Ref="#PWR019"  Part="1"
+F 0 "#PWR021" H 1750 2250 40  0001 C CNN
 F 1 "AGND" H 1750 2180 50  0000 C CNN
 	1    1750 2250

Commit message: Small fixes. The modular-half-dual board is final now.
Changed lines of the file:
@@
-EESchema Schematic File Version 2  date Sat 26 May 2012 12:20:03 PM CEST
+EESchema Schematic File Version 2  date Sat 28 Jul 2012 05:10:15 PM CEST
 LIBS:power
 LIBS:device
@@
 Sheet 2 6
 Title ""
-Date "26 may 2012"
+Date "28 jul 2012"
 Rev ""
 Comp ""
@@
 AR Path="/4FBE6CF5/4FBE6C5A" Ref="J7"  Part="1"
 AR Path="/4FBE6CE5/4FBE6C5A" Ref="J5"  Part="1"
-F 0 "J5" H 1775 1715 60  0000 C CNN
+F 0 "J3" H 1775 1715 60  0000 C CNN
 F 1 "SMA" H 1840 1640 60  0000 C CNN
 F 2 "SMA" H 1825 1570 50  0000 C CNN
@@
 AR Path="/4FBE6CF5/4FBE6C59" Ref="J8"  Part="1"
 AR Path="/4FBE6CE5/4FBE6C59" Ref="J6"  Part="1"
-F 0 "J6" H 1775 2515 60  0000 C CNN
+F 0 "J4" H 1775 2515 60  0000 C CNN
 F 1 "SMA" H 1840 2440 60  0000 C CNN
 F 2 "SMA" H 1825 2370 50  0000 C CNN
@@
 AR Path="/4FBE6CF5/4FBE6C58" Ref="R60"  Part="1"
 AR Path="/4FBE6CE5/4FBE6C58" Ref="R58"  Part="1"
-F 0 "R58" V 2230 1700 50  0000 C CNN
+F 0 "R56" V 2230 1700 50  0000 C CNN
 F 1 "20k" V 2150 1700 50  0000 C CNN
 	1    2150 1700
@@
 AR Path="/4FBE6CF5/4FBE6C57" Ref="R61"  Part="1"
 AR Path="/4FBE6CE5/4FBE6C57" Ref="R59"  Part="1"
-F 0 "R59" V 2230 1900 50  0000 C CNN
+F 0 "R57" V 2230 1900 50  0000 C CNN
 F 1 "20k" V 2150 1900 50  0000 C CNN
 	1    2150 1900
@@
 $EndComp
 $Comp
-L AGND #PWR020
+L AGND #PWR22
 U 1 1 4FBE6C56
 P 1850 1550
-AR Path="/4FBE6C46/4FBE6C56" Ref="#PWR020"  Part="1"
+AR Path="/4FBE6C46/4FBE6C56" Ref="#PWR22"  Part="1"
 AR Path="/4FBE6CFE/4FBE6C56" Ref="#PWR013"  Part="1"
 AR Path="/4FBE6CF5/4FBE6C56" Ref="#PWR015"  Part="1"
-AR Path="/4FBE6CE5/4FBE6C56" Ref="#PWR018"  Part="1"
-F 0 "#PWR020" H 1850 1550 40  0001 C CNN
+AR Path="/4FBE6CE5/4FBE6C56" Ref="#PWR20"  Part="1"
+F 0 "#PWR22" H 1850 1550 40  0001 C CNN
 F 1 "AGND" H 1850 1480 50  0000 C CNN
 	1    1850 1550
@@
 $EndComp
 $Comp
-L AGND #PWR021
+L AGND #PWR21
 U 1 1 4FBE6C55
 P 1750 2250
-AR Path="/4FBE6C46/4FBE6C55" Ref="#PWR021"  Part="1"
+AR Path="/4FBE6C46/4FBE6C55" Ref="#PWR21"  Part="1"
 AR Path="/4FBE6CFE/4FBE6C55" Ref="#PWR014"  Part="1"
 AR Path="/4FBE6CF5/4FBE6C55" Ref="#PWR016"  Part="1"
-AR Path="/4FBE6CE5/4FBE6C55" Ref="#PWR019"  Part="1"
-F 0 "#PWR021" H 1750 2250 40  0001 C CNN
+AR Path="/4FBE6CE5/4FBE6C55" Ref="#PWR19"  Part="1"
+F 0 "#PWR21" H 1750 2250 40  0001 C CNN
 F 1 "AGND" H 1750 2180 50  0000 C CNN
 	1    1750 2250
