File: modular-half-dual.sch (KiCad schematic (older format))
At the start: 18 parts, among them J1 SMA, J2 SMA, U1 TL071

Commit message: Finished the two-channel dual ti afe/pure analog-arduino adc version.
Parts:
- removed J1: SMA, SMA, symbol SMA
- added 20k1: 20k, symbol R
- added D1, D2: LED, symbol LED
- added P1, P3: CONN_4, symbol CONN_4
- added P10, P11, P12, P13, P14, P5, P6, P7, P8, P9: CONN_1, symbol CONN_1
- added R8: R, symbol R
- R4: value 20k -> R
Connections:
- net labels added: ar2, ar3, ar4, ar7, ar8, ar9, cs, drdy
- net labels removed: ch3, ch3n, ch3p, ch4, ch4n, ch4p, cs2, drdy1, drdy2
- wire segments 84 -> 73
- no-connect marks 3 -> 1
Other:
- note added: "extension connector 1"

Commit message: Added split ground planes
Parts:
- removed P10: CONN_1, symbol CONN_1
Changed lines of the file:
@@
-EESchema Schematic File Version 2  date Fri 25 May 2012 10:34:43 PM CEST
+EESchema Schematic File Version 2  date Sat 26 May 2012 12:20:03 PM CEST
 LIBS:power
 LIBS:device
@@
 Sheet 1 6
 Title ""
-Date "25 may 2012"
+Date "26 may 2012"
 Rev ""
 Comp ""
@@
 Comment4 ""
 $EndDescr
+$Comp
+L DGND #PWR?
+U 1 1 4FC0AE50
+P 5200 1800
+F 0 "#PWR?" H 5200 1800 40  0001 C CNN
+F 1 "DGND" H 5200 1730 40  0000 C CNN
+	1    5200 1800
+	0    -1   -1   0
+$EndComp
 $Comp
 L AGND #PWR01
@@
 ar4
 $Comp
-L CONN_1 P10
-U 1 1 4FBFB0CC
-P 5350 1800
-F 0 "P10" H 5430 1800 40  0000 L CNN
-F 1 "CONN_1" H 5350 1855 30  0001 C CNN
-	1    5350 1800
-	1    0    0    -1
-$EndComp
-$Comp
 L CONN_1 P9

Commit message: Small fixes. The modular-half-dual board is final now.
Parts:
- removed P12, P13, P5, P6, P9: CONN_1, symbol CONN_1
- added P2: CONN_1, symbol CONN_1
Connections:
- wire segments 73 -> 68
Changed lines of the file:
@@
-EESchema Schematic File Version 2  date Sat 26 May 2012 12:20:03 PM CEST
+EESchema Schematic File Version 2  date Sat 28 Jul 2012 05:10:15 PM CEST
 LIBS:power
 LIBS:device
@@
 Sheet 1 6
 Title ""
-Date "26 may 2012"
+Date "28 jul 2012"
 Rev ""
 Comp ""
@@
 Comment4 ""
 $EndDescr
-$Comp
-L DGND #PWR?
+Connection ~ 3300 2300
+$Comp
+L CONN_1 P2
+U 1 1 5013FFD5
+P 8650 1250
+F 0 "P2" H 8730 1250 40  0000 L CNN
+F 1 "CONN_1" H 8650 1305 30  0001 C CNN
+	1    8650 1250
+	0    -1   -1   0
+$EndComp
+$Comp
+L DGND #PWR8
 U 1 1 4FC0AE50
 P 5200 1800
-F 0 "#PWR?" H 5200 1800 40  0001 C CNN
+F 0 "#PWR8" H 5200 1800 40  0001 C CNN
 F 1 "DGND" H 5200 1730 40  0000 C CNN
 	1    5200 1800
@@
 $EndComp
 $Comp
-L AGND #PWR01
+L AGND #PWR14
 U 1 1 4FBFEB71
 P 7850 2650
-F 0 "#PWR01" H 7850 2650 40  0001 C CNN
+F 0 "#PWR14" H 7850 2650 40  0001 C CNN
 F 1 "AGND" H 7850 2580 50  0000 C CNN
 	1    7850 2650
@@
 $EndComp
 $Comp
-L AGND #PWR02
+L AGND #PWR18
 U 1 1 4FBFEB6D
 P 9000 2650
-F 0 "#PWR02" H 9000 2650 40  0001 C CNN
+F 0 "#PWR18" H 9000 2650 40  0001 C CNN
 F 1 "AGND" H 9000 2580 50  0000 C CNN
 	1    9000 2650
@@
 AVCC
 Wire Wire Line
-	5200 3300 5150 3300
-Wire Wire Line
 	5150 3100 5500 3100
 Wire Wire Line
@@
 Wire Wire Line
 	5500 2400 5150 2400
-Wire Wire Line
-	3250 2100 3200 2100
-Wire Wire Line
-	5150 1700 5200 1700
 Wire Wire Line
 	2850 5200 2850 5150
@@
 	5150 1800 5200 1800
 Wire Wire Line
-	3250 2600 3200 2600
-Wire Wire Line
 	5500 2300 5150 2300
 Wire Wire Line
@@
 Wire Wire Line
 	5500 3000 5150 3000
-Wire Wire Line
-	5200 3200 5150 3200
-$Comp
-L CONN_1 P13
-U 1 1 4FBFD87D
-P 5350 3300
-F 0 "P13" H 5430 3300 40  0000 L CNN
-F 1 "CONN_1" H 5350 3355 30  0001 C CNN
-	1    5350 3300
-	1    0    0    -1
-$EndComp
-$Comp
-L CONN_1 P12
-U 1 1 4FBFD879
-P 5350 3200
-F 0 "P12" H 5430 3200 40  0000 L CNN
-F 1 "CONN_1" H 5350 3255 30  0001 C CNN
-	1    5350 3200
-	1    0    0    -1
-$EndComp
 Text Label 5500 2300 2    60   ~ 0
 ar9
@@
 ar4
 $Comp
-L CONN_1 P9
-U 1 1 4FBFB0C9
-P 5350 1700
-F 0 "P9" H 5430 1700 40  0000 L CNN
-F 1 "CONN_1" H 5350 1755 30  0001 C CNN
-	1    5350 1700
-	1    0    0    -1
-$EndComp
-$Comp
-L CONN_1 P5
-U 1 1 4FBFB0EB
-P 3050 2100
-F 0 "P5" H 3130 2100 40  0000 L CNN
-F 1 "CONN_1" H 3050 2155 30  0001 C CNN
-	1    3050 2100
-	-1   0    0    1
-$EndComp
-$Comp
-L CONN_1 P6
-U 1 1 4FBFB0E8
-P 3050 2600
-F 0 "P6" H 3130 2600 40  0000 L CNN
-F 1 "CONN_1" H 3050 2655 30  0001 C CNN
-	1    3050 2600
-	-1   0    0    1
-$EndComp
-$Comp
-L DGND #PWR03
+L DGND #PWR2
 U 1 1 4FBFAA0E
 P 3100 6100
-F 0 "#PWR03" H 3100 6100 40  0001 C CNN
+F 0 "#PWR2" H 3100 6100 40  0001 C CNN
 F 1 "DGND" H 3100 6030 40  0000 C CNN
 	1    3100 6100
@@
 $EndComp
 $Comp
-L DGND #PWR04
+L DGND #PWR1
 U 1 1 4FBFAA0B
 P 2850 6100
-F 0 "#PWR04" H 2850 6100 40  0001 C CNN
+F 0 "#PWR1" H 2850 6100 40  0001 C CNN
 F 1 "DGND" H 2850 6030 40  0000 C CNN
 	1    2850 6100
@@
 $EndComp
 $Comp
-L AGND #PWR05
+L AGND #PWR13
 U 1 1 4FBFA30F
 P 7850 2450
-F 0 "#PWR05" H 7850 2450 40  0001 C CNN
+F 0 "#PWR13" H 7850 2450 40  0001 C CNN
 F 1 "AGND" H 7850 2380 50  0000 C CNN
 	1    7850 2450
@@
 $EndComp
 $Comp
-L AGND #PWR06
+L AGND #PWR17
 U 1 1 4FBFA30B
 P 9000 2450
-F 0 "#PWR06" H 9000 2450 40  0001 C CNN
+F 0 "#PWR17" H 9000 2450 40  0001 C CNN
 F 1 "AGND" H 9000 2380 50  0000 C CNN
 	1    9000 2450
@@
 pwdn
 $Comp
-L DGND #PWR07
+L DGND #PWR10
 U 1 1 4FBF8780
 P 6150 1250
-F 0 "#PWR07" H 6150 1250 40  0001 C CNN
+F 0 "#PWR10" H 6150 1250 40  0001 C CNN
 F 1 "DGND" H 6150 1180 40  0000 C CNN
 	1    6150 1250
@@
 $EndComp
 $Comp
-L AGND #PWR08
+L AGND #PWR9
 U 1 1 4FBF877C
 P 5800 1250
-F 0 "#PWR08" H 5800 1250 40  0001 C CNN
+F 0 "#PWR9" H 5800 1250 40  0001 C CNN
 F 1 "AGND" H 5800 1180 50  0000 C CNN
 	1    5800 1250
@@
 $EndComp
 $Comp
-L AGND #PWR09
+L AGND #PWR11
 U 1 1 4FBE929C
 P 7050 1800
-F 0 "#PWR09" H 7050 1800 40  0001 C CNN
+F 0 "#PWR11" H 7050 1800 40  0001 C CNN
 F 1 "AGND" H 7050 1730 50  0000 C CNN
 	1    7050 1800
@@
 AVCC
 $Comp
-L AGND #PWR010
+L AGND #PWR12
 U 1 1 4FBE928A
 P 7850 1800
-F 0 "#PWR010" H 7850 1800 40  0001 C CNN
+F 0 "#PWR12" H 7850 1800 40  0001 C CNN
 F 1 "AGND" H 7850 1730 50  0000 C CNN
 	1    7850 1800
@@
 $EndComp
 $Comp
-L AGND #PWR011
+L AGND #PWR16
 U 1 1 4FBE9288
 P 8650 1800
-F 0 "#PWR011" H 8650 1800 40  0001 C CNN
+F 0 "#PWR16" H 8650 1800 40  0001 C CNN
 F 1 "AGND" H 8650 1730 50  0000 C CNN
 	1    8650 1800
@@
 $EndComp
 $Comp
-L DGND #PWR012
+L DGND #PWR7
 U 1 1 4FBE8DDB
 P 4850 1200
-F 0 "#PWR012" H 4850 1200 40  0001 C CNN
+F 0 "#PWR7" H 4850 1200 40  0001 C CNN
 F 1 "DGND" H 4850 1130 40  0000 C CNN
 	1    4850 1200
@@
 $EndComp
 $Comp
-L DGND #PWR013
+L DGND #PWR3
 U 1 1 4FBE8DD5
 P 3200 2400
-F 0 "#PWR013" H 3200 2400 40  0001 C CNN
+F 0 "#PWR3" H 3200 2400 40  0001 C CNN
 F 1 "DGND" H 3200 2330 40  0000 C CNN
 	1    3200 2400
@@
 $EndComp
 $Comp
-L AGND #PWR014
+L AGND #PWR15
 U 1 1 4FBE6B97
 P 7950 4700
-F 0 "#PWR014" H 7950 4700 40  0001 C CNN
+F 0 "#PWR15" H 7950 4700 40  0001 C CNN
 F 1 "AGND" H 7950 4630 50  0000 C CNN
 	1    7950 4700
@@
 $EndSheet
 $Comp
-L AGND #PWR015
+L AGND #PWR5
 U 1 1 4FB7BF15
 P 3750 1200
-F 0 "#PWR015" H 3750 1200 40  0001 C CNN
+F 0 "#PWR5" H 3750 1200 40  0001 C CNN
 F 1 "AGND" H 3750 1130 50  0000 C CNN
 	1    3750 1200
@@
 AVcc
 $Comp
-L +5V #PWR016
+L +5V #PWR4
 U 1 1 4FB7BEF6
 P 3250 2300
-F 0 "#PWR016" H 3250 2390 20  0001 C CNN
+F 0 "#PWR4" H 3250 2390 20  0001 C CNN
 F 1 "+5V" H 3250 2390 30  0000 C CNN
 	1    3250 2300
@@
 $EndComp
 $Comp
-L +5V #PWR017
+L +5V #PWR6
 U 1 1 4FB7BEF0
 P 4800 800
-F 0 "#PWR017" H 4800 890 20  0001 C CNN
+F 0 "#PWR6" H 4800 890 20  0001 C CNN
 F 1 "+5V" H 4800 890 30  0000 C CNN
 	1    4800 800
